Commit message: Add files via upload

File: compass_gait_walker/urdf/compass_gait_walker.urdf (robot description, URDF)
Before this commit: robot compass_gait_walker, 3 links, 2 joints
Links:
- removed link left_leg_Link
- removed link right_leg_Link
- added link left_leg_link, mass 5; collision mesh filename=package://compass_gait_walker/meshes/left_leg_link.STL; visual mesh filename=package://compass_gait_walker/meshes/left_leg_link.STL
- added link right_leg_link, mass 5; collision mesh filename=package://compass_gait_walker/meshes/right_leg_link.STL; visual mesh filename=package://compass_gait_walker/meshes/right_leg_link.STL
Joints:
- joint left_leg_joint: axis 0 1 0 -> 0 -1 0; child left_leg_Link -> left_leg_link; limit lower=0 upper=0 effort=0 velocity=0 -> lower=-1.57 upper=1.57 effort=100 velocity=100; origin xyz=0.0078635 -0.11 -0.49994 rpy=0 -0.015728 0 -> xyz=0 -0.12 -0.5 rpy=0 0 0
- joint right_leg_joint: axis 0 1 0 -> 0 -1 0; child right_leg_Link -> right_leg_link; limit lower=0 upper=0 effort=0 velocity=0 -> lower=-1.57 upper=1.57 effort=100 velocity=100; origin xyz=0.0078635 0.1 -0.49994 rpy=0 -0.015728 0 -> xyz=0 0.12 -0.5 rpy=0 0 0
